File: KiCAD/LED Board/LED Board.kicad_pcb (KiCad board)
At the start: 2 copper layers, 203.2 x 254 mm, 25 parts, among them J1 Conn_01x03_Socket, J10 Conn_01x03_Socket, J2 Conn_01x03_Socket, J3 Conn_01x03_Socket, J4 Conn_01x03_Socket, J5 Conn_01x03_Socket, J6 Conn_01x03_Socket, J7 Conn_01x03_Socket, J8 Conn_01x03_Socket, J9 Conn_01x03_Socket

Commit message: Updated LED Socket Board
Parts:
- removed the J1 at (209.6, 252.2)
- removed the J10 at (209.6, 137.9)
- removed the J2 at (209.6, 239.5)
- removed the J3 at (209.6, 226.8)
- removed the J4 at (209.6, 214.1)
- removed the J5 at (209.6, 201.4)
- removed the J6 at (209.6, 188.7)
- removed the J7 at (209.6, 176.0)
- removed the J8 at (209.6, 163.3)
- removed the J9 at (209.6, 150.6)
- added CTRL_OUT1: Conn_01x03_Socket, CustomConnectorPinSocket2.54mm1x03_Vertical:PinSocket_1x03_P2.54mm_Vertical_HandSolder, F.Cu at (56.5, 100.0)
- added J11: Conn_01x03_Socket, CustomConnectorPinSocket2.54mm1x03_Vertical:PinSocket_1x03_P2.54mm_Vertical_HandSolder, F.Cu at (224.5, 125.0)
- added J12: Conn_01x03_Socket, CustomConnectorPinSocket2.54mm1x03_Vertical:PinSocket_1x03_P2.54mm_Vertical_HandSolder, F.Cu at (224.5, 153.2)
- added J13: Conn_01x03_Socket, CustomConnectorPinSocket2.54mm1x03_Vertical:PinSocket_1x03_P2.54mm_Vertical_HandSolder, F.Cu at (224.5, 139.1)
- added J14: Conn_01x03_Socket, CustomConnectorPinSocket2.54mm1x03_Vertical:PinSocket_1x03_P2.54mm_Vertical_HandSolder, F.Cu at (224.5, 167.3)
- added J15: Conn_01x03_Socket, CustomConnectorPinSocket2.54mm1x03_Vertical:PinSocket_1x03_P2.54mm_Vertical_HandSolder, F.Cu at (224.5, 181.4)
- added J16: Conn_01x03_Socket, CustomConnectorPinSocket2.54mm1x03_Vertical:PinSocket_1x03_P2.54mm_Vertical_HandSolder, F.Cu at (224.5, 195.6)
- added J17: Conn_01x03_Socket, CustomConnectorPinSocket2.54mm1x03_Vertical:PinSocket_1x03_P2.54mm_Vertical_HandSolder, F.Cu at (224.5, 209.7)
- added J18: Conn_01x03_Socket, CustomConnectorPinSocket2.54mm1x03_Vertical:PinSocket_1x03_P2.54mm_Vertical_HandSolder, F.Cu at (224.5, 223.8)
- added J19: Conn_01x03_Socket, CustomConnectorPinSocket2.54mm1x03_Vertical:PinSocket_1x03_P2.54mm_Vertical_HandSolder, F.Cu at (224.5, 237.9)
- added J20: Conn_01x03_Socket, CustomConnectorPinSocket2.54mm1x03_Vertical:PinSocket_1x03_P2.54mm_Vertical_HandSolder, F.Cu at (224.5, 252.0)
- CTRL_IN1, J1, J10, J2, J3, J4, J5, J6, J7, J8, J9: footprint Connector_PinSocket_2.54mm:PinSocket_1x03_P2.54mm_Vertical -> CustomConnectorPinSocket2.54mm1x03_Vertical:PinSocket_1x03_P2.54mm_Vertical_HandSolder
- moved CTRL_IN1 20.0 mm to (56.5, 306.9)
- moved J10 16.0 mm to (56.5, 125.0)
- moved J9 14.5 mm to (56.5, 139.7)
- moved J8 13.0 mm to (56.5, 154.5)
- moved J7 11.7 mm to (56.5, 169.2)
- moved J1 10.9 mm to (56.5, 257.6)
- moved J6 10.6 mm to (56.5, 183.9)
- moved J2 10.1 mm to (56.5, 242.8)
- moved J5 9.90 mm to (56.5, 198.7)
- moved J3 9.59 mm to (56.5, 228.1)
- moved J4 9.53 mm to (56.5, 213.4)
Routing:
- net /DIN: track 181.5 -> 221.1 mm
Other:
- board text added: "CTRL_IN"
- board text added: "CTRL_OUT"
- board text added: "DOUT"
- board text added: "VOUT"
